Commit message: first try move gripper in gazebo

File: earth_ws/src/dodo_arm_pkg/urdf/dodo_arm_realsense.xacro (robot description, xacro)
@@ -61,8 +61,8 @@
 	    <type>transmission_interface/SimpleTransmission</type>
 	    <joint name="${joint_name}">
-	      <hardwareInterface>hardware_interface/PositionJointInterface</hardwareInterface>
+	      <hardwareInterface>hardware_interface/EffortJointInterface</hardwareInterface>
 	    </joint>
 	    <actuator name="motor1">
-	      <hardwareInterface>hardware_interface/PositionJointInterface</hardwareInterface>
+	      <hardwareInterface>hardware_interface/EffortJointInterface</hardwareInterface>
 	      <mechanicalReduction>1</mechanicalReduction>
 	    </actuator>
@@ -175,37 +175,8 @@
     <material>Gazebo/White</material>
   </gazebo>
-  <joint name="elbow_roll_joint" type="fixed">
+  <joint name="elbow_pitch_joint" type="revolute">
     <parent link="shoulder_pitch_link"/>
-    <child link="elbow_roll_link"/>
-    <origin xyz="-0.002 0 0.1206" rpy="${M_PI} ${M_PI/2} 0" />
-    <axis xyz="-1 0 0" />
-    <limit effort="300" velocity="1" lower="-2.61799387799" upper="0.705631162427" />
-    <dynamics damping="50" friction="1"/>
-  </joint>
-<!-- ///////////////////////////////////////////////////////////////////////////////////////////////////////////////////// -->
-  <!-- ELBOW ROLL LINK -->
-  <link name="elbow_roll_link" >
-    <visual>
-      <origin xyz="-0.015 0.0 -0.0" rpy="0 ${M_PI/2} 0" />
-      <geometry>
-            <cylinder radius="${elbow_roll_width}" length="${elbow_roll_len}"/>
-      </geometry>
-      <material name="Black" />
-    </visual>
-    <collision>
-      <origin xyz="-0.015 0.0 -0.0" rpy="0 ${M_PI/2} 0" />
-      <geometry>
-            <cylinder radius="${elbow_roll_width}" length="${elbow_roll_len}"/>
-      </geometry>
-    </collision>
-	<xacro:inertial_matrix mass="1"/>
-  </link>
-  <gazebo reference="elbow_roll_link">
-    <material>Gazebo/Black</material>
-  </gazebo>
-  <joint name="elbow_pitch_joint" type="revolute">
-    <parent link="elbow_roll_link"/>
     <child link="elbow_pitch_link"/>
-    <origin xyz="-0.035 0 0.0" rpy="0.055 ${M_PI/2} 0" />
+    <origin xyz="-0.002 0 0.10" rpy="0.055 ${M_PI} 0" />
     <axis xyz="1 0 0" />
     <limit effort="300" velocity="1" lower="-1.5953400194" upper="1.93281579274" />
@@ -406,5 +377,4 @@
    <xacro:transmission_block joint_name="shoulder_pan_joint"/>
    <xacro:transmission_block joint_name="shoulder_pitch_joint"/>
-   <xacro:transmission_block joint_name="elbow_roll_joint"/>
    <xacro:transmission_block joint_name="elbow_pitch_joint"/>
    <xacro:transmission_block joint_name="wrist_roll_joint"/>
