Commit message: success pick place box panda_moveit_config

File: earth_ws/src/panda_moveit_config/config/panda_arm_hand.srdf.xacro (robot description, xacro)
@@ -19,5 +19,5 @@
   </group>
   <!--GROUP STATES: Purpose: Define a named state for a particular group, in terms of joint values. This is useful to define states like 'folded arms'-->
-  <!-- <group_state name="ready" group="panda_arm_hand">
+  <group_state name="ready" group="panda_arm_hand">
     <joint name="panda_joint1" value="0" />
     <joint name="panda_joint2" value="-0.785" />
@@ -27,5 +27,7 @@
     <joint name="panda_joint6" value="1.571" />
     <joint name="panda_joint7" value="0.785" />
-  </group_state> -->
+    <joint name="panda_finger_joint1" value="0.04" />
+    <joint name="panda_finger_joint2" value="0.04" />
+  </group_state>
   <!--END EFFECTOR: Purpose: Represent information about an end effector.-->
   <end_effector name="hand" parent_link="panda_link8" group="hand" parent_group="panda_arm_hand" />
