Commit message: add cr3_moveit_3

File: cr3_ws/src/tesr_ros_cr3_pkg/urdf/cr3_robot_w_gripper_seperated.xacro (robot description, xacro)
@@ -16,8 +16,8 @@
       <type>transmission_interface/SimpleTransmission</type>
       <joint name="${joint}">
-        <hardwareInterface>hardware_interface/PositionJointInterface</hardwareInterface>
+        <hardwareInterface>hardware_interface/EffortJointInterface</hardwareInterface>
       </joint>
       <actuator name="${motor}">
-        <hardwareInterface>hardware_interface/PositionJointInterface</hardwareInterface>
+        <hardwareInterface>hardware_interface/EffortJointInterface</hardwareInterface>
         <mechanicalReduction>1</mechanicalReduction>
       </actuator>
@@ -39,5 +39,5 @@
     </visual>
     <collision>
-      <origin xyz="0 0 0" rpy="0 0 0" />
+      <origin xyz="0 0 0" rpy="0 0 -1.57" />
       <geometry>
         <mesh filename="package://tesr_ros_cr3_pkg/meshes/base_link.STL" />
@@ -48,4 +48,5 @@
     <parent link="world" />
     <child link="base_link" />
+    <origin xyz="0.0 0.0 0.0" rpy="0.0 0.0 0.0" />
   </joint>
   <link name="Link1">
@@ -205,5 +206,5 @@
   <joint name="joint6" type="revolute">
     <origin xyz="0 0.105 0" rpy="-1.5708 0 0" />
-    <parent link="Link5" />
+    <parent link="Link5" />d
     <child link="Link6" />
     <axis xyz="0 0 1" />
@@ -211,8 +212,8 @@
     <dynamics damping="1.0" />
   </joint>
-  <link name="Gripper">
-    <inertial>
-      <origin xyz="0 0 0" rpy="0 0 0" />
-      <mass value="0.95" />
+  <link name="hand">
+    <inertial>
+      <origin xyz="0 0 0" rpy="0 0 0" />
+      <mass value="0.75" />
       <inertia ixx="0.0" ixy="0.0" ixz="0.0" iyy="0.0" iyz="0.0" izz="0.0" />
     </inertial>
@@ -232,10 +233,10 @@
   <joint name="joint7" type="fixed">
     <parent link="Link6" />
-    <child link="Gripper" />
-  </joint>
-  <link name="FingerL">
-    <inertial>
-      <origin xyz="0 0 0" rpy="0 0 0" />
-      <mass value="0.95" />
+    <child link="hand" />
+  </joint>
+  <link name="finger_l">
+    <inertial>
+      <origin xyz="0 0 0" rpy="0 0 0" />
+      <mass value="0.10" />
       <inertia ixx="0.0" ixy="0.0" ixz="0.0" iyy="0.0" iyz="0.0" izz="0.0" />
     </inertial>
@@ -247,5 +248,5 @@
     </visual>
     <collision>
-      <origin xyz="0.053 0.035 0.05" rpy="1.54 0 0" />
+      <origin xyz="0.053 0.035 -0.015" rpy="1.54 0 0" />
       <geometry>
         <mesh filename="package://tesr_ros_cr3_pkg/meshes/FingerL.stl" scale="0.0008 0.0008 0.0008" />
@@ -253,15 +254,15 @@
     </collision>
   </link>
-  <joint name="joint8" type="prismatic">
-    <parent link="Gripper" />
-    <child link="FingerL" />
+  <joint name="joint8" type="revolute">
+    <parent link="hand" />
+    <child link="finger_l" />
     <origin rpy="0 0 0" xyz="0 0 0.0584"/>
-    <axis xyz="1 0 0"/>
+    <axis xyz="0 0 1"/>
     <limit effort="20" lower="0.0" upper="0.04" velocity="0.2"/>
   </joint>
-  <link name="FingerR">
-    <inertial>
-      <origin xyz="0 0 0" rpy="0 0 0" />
-      <mass value="0.95" />
+  <link name="finger_r">
+    <inertial>
+      <origin xyz="0 0 0" rpy="0 0 0" />
+      <mass value="0.15" />
       <inertia ixx="0.0" ixy="0.0" ixz="0.0" iyy="0.0" iyz="0.0" izz="0.0" />
     </inertial>
@@ -273,5 +274,5 @@
     </visual>
     <collision>
-      <origin xyz="0.053 0.035 0.05" rpy="1.54 0 0" />
+      <origin xyz="0.053 0.035 -0.015" rpy="1.54 0 0" />
       <geometry>
         <mesh filename="package://tesr_ros_cr3_pkg/meshes/FingerR v1.stl" scale="0.0008 0.0008 0.0008" />
@@ -279,9 +280,9 @@
     </collision>
   </link>
-  <joint name="joint9" type="prismatic">
-    <parent link="Gripper" />
-    <child link="FingerR" />
+  <joint name="joint9" type="revolute">
+    <parent link="hand" />
+    <child link="finger_r" />
     <origin rpy="0 0 0" xyz="0 0 0.0584"/>
-    <axis xyz="-1 0 0"/>
+    <axis xyz="0 0 -1"/>
     <limit effort="20" lower="0.0" upper="0.04" velocity="0.2"/>
   </joint>
@@ -305,4 +306,4 @@
         <xacro:arm_gazebo link="link5"/>
         <xacro:arm_gazebo link="link6"/>
-        <xacro:arm_gazebo link="Gripper"/>
+        <xacro:arm_gazebo link="hand"/>
 </robot>

Commit message: finished cr3_moveit_3

File: cr3_ws/src/tesr_ros_cr3_pkg/urdf/cr3_robot_w_gripper_seperated.xacro (robot description, xacro)
@@ -4,5 +4,6 @@
      For more information, please see http://wiki.ros.org/sw_urdf_exporter -->
 <robot xmlns:xacro="http://www.ros.org/wiki/xacro" name="cr3_robot">
-  <!-- xacro macro-->
+  <!-- <xacro:property name="damping_value" value="0" />
+  <xacro:property name="friction_value" value="0.5" /> -->
   <xacro:macro name="arm_gazebo" params="link">
             <gazebo reference="${link}">
@@ -16,8 +17,8 @@
       <type>transmission_interface/SimpleTransmission</type>
       <joint name="${joint}">
-        <hardwareInterface>hardware_interface/EffortJointInterface</hardwareInterface>
+        <hardwareInterface>hardware_interface/PositionJointInterface</hardwareInterface>
       </joint>
       <actuator name="${motor}">
-        <hardwareInterface>hardware_interface/EffortJointInterface</hardwareInterface>
+        <hardwareInterface>hardware_interface/PositionJointInterface</hardwareInterface>
         <mechanicalReduction>1</mechanicalReduction>
       </actuator>
@@ -74,6 +75,6 @@
     <child link="Link1" />
     <axis xyz="0 0 1" />
-    <limit lower="-3.14" upper="3.14" effort="0" velocity="0" />
-    <dynamics damping="1.0" />
+    <limit lower="-3.14" upper="3.14" effort="1000" velocity="100" />
+    <!-- <dynamics damping="${damping_value}" friction="${friction_value}"/> -->
   </joint>
   <link name="Link2">
@@ -101,6 +102,6 @@
     <child link="Link2" />
     <axis xyz="0 0 1" />
-    <limit lower="-3.14" upper="3.14" effort="0" velocity="0" />
-    <dynamics damping="1.0" />
+    <limit lower="-3.14" upper="3.14" effort="1000" velocity="100" />
+    <!-- <dynamics damping="${damping_value}" friction="${friction_value}"/> -->
   </joint>
   <link name="Link3">
@@ -128,6 +129,6 @@
     <child link="Link3" />
     <axis xyz="0 0 1" />
-    <limit lower="-3.14" upper="3.14" effort="0" velocity="0" />
-    <dynamics damping="1.0" />
+    <limit lower="-3.14" upper="3.14" effort="1000" velocity="100" />
+     <!-- <dynamics damping="${damping_value}" friction="${friction_value}"/> -->
   </joint>
   <link name="Link4">
@@ -155,6 +156,6 @@
     <child link="Link4" />
     <axis xyz="0 0 1" />
-    <limit lower="-3.14" upper="3.14" effort="0" velocity="0" />
-    <dynamics damping="1.0" />
+    <limit lower="-3.14" upper="3.14" effort="1000" velocity="100" />
+    <!-- <dynamics damping="${damping_value}" friction="${friction_value}"/> -->
   </joint>
   <link name="Link5">
@@ -182,6 +183,6 @@
     <child link="Link5" />
     <axis xyz="0 0 1" />
-    <limit lower="-3.14" upper="3.14" effort="0" velocity="0" />
-    <dynamics damping="1.0" />
+    <limit lower="-3.14" upper="3.14" effort="1000" velocity="100" />
+    <!-- <dynamics damping="${damping_value}" friction="${friction_value}"/> -->
   </joint>
   <link name="Link6">
@@ -209,12 +210,12 @@
     <child link="Link6" />
     <axis xyz="0 0 1" />
-    <limit lower="-3.14" upper="3.14" effort="0" velocity="0" />
-    <dynamics damping="1.0" />
+    <limit lower="-3.14" upper="3.14" effort="1000" velocity="100" />
+    <!-- <dynamics damping="${damping_value}" friction="${friction_value}"/> -->
   </joint>
   <link name="hand">
     <inertial>
       <origin xyz="0 0 0" rpy="0 0 0" />
-      <mass value="0.75" />
-      <inertia ixx="0.0" ixy="0.0" ixz="0.0" iyy="0.0" iyz="0.0" izz="0.0" />
+      <mass value="0.6" />
+      <inertia ixx="0.1" ixy="0.0" ixz="0.0" iyy="0.1" iyz="0.0" izz="0.1" />
     </inertial>
     <visual>
@@ -227,5 +228,5 @@
       <origin xyz="0.053 0.035 0.05" rpy="1.54 0 0" />
       <geometry>
-        <mesh filename="package://tesr_ros_cr3_pkg/meshes/base_gripper.stl" scale="0.0008 0.0008 0.0008" />
+        <mesh filename="package://tesr_ros_cr3_pkg/meshes/base_gripper.stl" scale="0.001 0.001 0.001" />
       </geometry>
     </collision>
@@ -238,6 +239,6 @@
     <inertial>
       <origin xyz="0 0 0" rpy="0 0 0" />
-      <mass value="0.10" />
-      <inertia ixx="0.0" ixy="0.0" ixz="0.0" iyy="0.0" iyz="0.0" izz="0.0" />
+      <mass value="0.3" />
+      <inertia ixx="0.1" ixy="0.0" ixz="0.0" iyy="0.1" iyz="0.0" izz="0.1" />
     </inertial>
     <visual>
@@ -250,5 +251,5 @@
       <origin xyz="0.053 0.035 -0.015" rpy="1.54 0 0" />
       <geometry>
-        <mesh filename="package://tesr_ros_cr3_pkg/meshes/FingerL.stl" scale="0.0008 0.0008 0.0008" />
+        <mesh filename="package://tesr_ros_cr3_pkg/meshes/FingerL.stl" scale="0.001 0.001 0.001" />
       </geometry>
     </collision>
@@ -258,12 +259,12 @@
     <child link="finger_l" />
     <origin rpy="0 0 0" xyz="0 0 0.0584"/>
-    <axis xyz="0 0 1"/>
-    <limit effort="20" lower="0.0" upper="0.04" velocity="0.2"/>
+    <axis xyz="0 1 0"/>
+    <limit effort="1000" lower="-0.785" upper="0.0" velocity="0.2"/>
   </joint>
   <link name="finger_r">
     <inertial>
       <origin xyz="0 0 0" rpy="0 0 0" />
-      <mass value="0.15" />
-      <inertia ixx="0.0" ixy="0.0" ixz="0.0" iyy="0.0" iyz="0.0" izz="0.0" />
+      <mass value="0.6" />
+      <inertia ixx="0.1" ixy="0.0" ixz="0.0" iyy="0.1" iyz="0.0" izz="0.1" />
     </inertial>
     <visual>
@@ -276,5 +277,5 @@
       <origin xyz="0.053 0.035 -0.015" rpy="1.54 0 0" />
       <geometry>
-        <mesh filename="package://tesr_ros_cr3_pkg/meshes/FingerR v1.stl" scale="0.0008 0.0008 0.0008" />
+        <mesh filename="package://tesr_ros_cr3_pkg/meshes/FingerR v1.stl" scale="0.001 0.001 0.001" />
       </geometry>
     </collision>
@@ -284,6 +285,6 @@
     <child link="finger_r" />
     <origin rpy="0 0 0" xyz="0 0 0.0584"/>
-    <axis xyz="0 0 -1"/>
-    <limit effort="20" lower="0.0" upper="0.04" velocity="0.2"/>
+    <axis xyz="0 1 0"/>
+    <limit effort="1000" lower="0.0" upper="0.785" velocity="0.2"/>
   </joint>
   <!-- xacro implement-->
@@ -307,3 +308,5 @@
         <xacro:arm_gazebo link="link6"/>
         <xacro:arm_gazebo link="hand"/>
+        <xacro:arm_gazebo link="finger_l"/>
+        <xacro:arm_gazebo link="finger_r"/>
 </robot>

Commit message: update on camera in cr_3 gazebo

File: cr3_ws/src/tesr_ros_cr3_pkg/urdf/cr3_robot_w_gripper_seperated.xacro (robot description, xacro)
@@ -288,4 +288,11 @@
     <limit effort="1000" lower="0.0" upper="0.785" velocity="0.2"/>
   </joint>
+    <!-- for Depth Camera -->
+  <xacro:property name="deg_to_rad" value="0.01745329251994329577"/>
+  <xacro:include filename="$(find tesr_ros_cr3_pkg)/urdf/_d435.xacro"/>
+  <xacro:sensor_d435 name="sensor_d435" topics_ns="sensor_d435" parent="Link6">
+    <origin xyz="0.0 -0.1 0.0" rpy="1.57 -1.57 0"/>
+    <!-- <origin xyz="0 0 0" rpy="${-90.0 * deg_to_rad} 0 ${-90.0 * deg_to_rad}"/> -->
+  </xacro:sensor_d435>
   <!-- xacro implement-->
   <xacro:arm_control transmission="tran_1" joint="joint1" motor="motor_1" />

Commit message: reallign the cr3 hand

File: cr3_ws/src/tesr_ros_cr3_pkg/urdf/cr3_robot_w_gripper_seperated.xacro (robot description, xacro)
@@ -220,5 +220,5 @@
     </inertial>
     <visual>
-      <origin xyz="0.053 0.035 0.05" rpy="1.54 0 0" />
+      <origin xyz="0.010 0.065 0.05" rpy="1.54 0 0.77" />
       <geometry>
         <mesh filename="package://tesr_ros_cr3_pkg/meshes/base_gripper.stl" scale="0.001 0.001 0.001" />
@@ -226,5 +226,5 @@
     </visual>
     <collision>
-      <origin xyz="0.053 0.035 0.05" rpy="1.54 0 0" />
+      <origin xyz="0.053 0.035 0.05" rpy="1.54 0 0.77" />
       <geometry>
         <mesh filename="package://tesr_ros_cr3_pkg/meshes/base_gripper.stl" scale="0.001 0.001 0.001" />
@@ -243,5 +243,5 @@
     </inertial>
     <visual>
-      <origin xyz="0.053 0.035 -0.015" rpy="1.54 0 0" />
+      <origin xyz="0.0 0.05 -0.010" rpy="1.54 0 0.77" />
       <geometry>
         <mesh filename="package://tesr_ros_cr3_pkg/meshes/FingerL.stl" scale="0.001 0.001 0.001" />
@@ -249,5 +249,5 @@
     </visual>
     <collision>
-      <origin xyz="0.053 0.035 -0.015" rpy="1.54 0 0" />
+      <origin xyz="0.01 0.05 -0.010" rpy="1.54 0 0.77" />
       <geometry>
         <mesh filename="package://tesr_ros_cr3_pkg/meshes/FingerL.stl" scale="0.001 0.001 0.001" />
@@ -269,5 +269,5 @@
     </inertial>
     <visual>
-      <origin xyz="0.053 0.035 -0.015" rpy="1.54 0 0" />
+      <origin xyz="0.0050 0.070 -0.005" rpy="1.54 0 0.77" />
       <geometry>
         <mesh filename="package://tesr_ros_cr3_pkg/meshes/FingerR v1.stl" scale="0.001 0.001 0.001" />
@@ -275,5 +275,5 @@
     </visual>
     <collision>
-      <origin xyz="0.053 0.035 -0.015" rpy="1.54 0 0" />
+      <origin xyz="0.0050 0.070 -0.005" rpy="1.54 0 0.77" />
       <geometry>
         <mesh filename="package://tesr_ros_cr3_pkg/meshes/FingerR v1.stl" scale="0.001 0.001 0.001" />
@@ -292,5 +292,5 @@
   <xacro:include filename="$(find tesr_ros_cr3_pkg)/urdf/_d435.xacro"/>
   <xacro:sensor_d435 name="sensor_d435" topics_ns="sensor_d435" parent="Link6">
-    <origin xyz="0.0 -0.1 0.0" rpy="1.57 -1.57 0"/>
+    <origin xyz="0.031 -0.031 0.0" rpy="1.57 -1.57 0.77"/>
     <!-- <origin xyz="0 0 0" rpy="${-90.0 * deg_to_rad} 0 ${-90.0 * deg_to_rad}"/> -->
   </xacro:sensor_d435>

Commit message: update cr3 collision block

File: cr3_ws/src/tesr_ros_cr3_pkg/urdf/cr3_robot_w_gripper_seperated.xacro (robot description, xacro)
@@ -66,5 +66,5 @@
       <origin xyz="0 0 0" rpy="0 0 0" />
       <geometry>
-        <mesh filename="package://tesr_ros_cr3_pkg/meshes/Link1.STL" />
+        <mesh filename="package://tesr_ros_cr3_pkg/meshes/Link1.STL" scale="1.3 1.3 1.3"/>
       </geometry>
     </collision>
@@ -91,7 +91,7 @@
     </visual>
     <collision>
-      <origin xyz="0 0 0" rpy="0 0 0" />
-      <geometry>
-        <mesh filename="package://tesr_ros_cr3_pkg/meshes/Link2.STL" />
+      <origin xyz="0.025 0.0 -0.025" rpy="0 0 0" />
+      <geometry>
+        <mesh filename="package://tesr_ros_cr3_pkg/meshes/Link2.STL" scale="1.1 1.3 1.3" />
       </geometry>
     </collision>
@@ -118,7 +118,7 @@
     </visual>
     <collision>
-      <origin xyz="0 0 0" rpy="0 0 0" />
-      <geometry>
-        <mesh filename="package://tesr_ros_cr3_pkg/meshes/Link3.STL" />
+      <origin xyz="0.025 0 0.0" rpy="0 0 0" />
+      <geometry>
+        <mesh filename="package://tesr_ros_cr3_pkg/meshes/Link3.STL" scale="1.1 1.5 1.5"/>
       </geometry>
     </collision>
@@ -147,5 +147,5 @@
       <origin xyz="0 0 0" rpy="0 0 0" />
       <geometry>
-        <mesh filename="package://tesr_ros_cr3_pkg/meshes/Link4.STL" />
+        <mesh filename="package://tesr_ros_cr3_pkg/meshes/Link4.STL" scale="1.1 1.5 1.5"/>
       </geometry>
     </collision>
@@ -174,5 +174,5 @@
       <origin xyz="0 0 0" rpy="0 0 0" />
       <geometry>
-        <mesh filename="package://tesr_ros_cr3_pkg/meshes/Link5.STL" />
+        <mesh filename="package://tesr_ros_cr3_pkg/meshes/Link5.STL" scale="1.1 1.5 1.5"/>
       </geometry>
     </collision>
@@ -201,5 +201,5 @@
       <origin xyz="0 0 0" rpy="0 0 0" />
       <geometry>
-        <mesh filename="package://tesr_ros_cr3_pkg/meshes/Link6.STL" />
+        <mesh filename="package://tesr_ros_cr3_pkg/meshes/Link6.STL" scale="1 1 1"/>
       </geometry>
     </collision>
@@ -226,5 +226,5 @@
     </visual>
     <collision>
-      <origin xyz="0.053 0.035 0.05" rpy="1.54 0 0.77" />
+      <origin xyz="0.010 0.065 0.05" rpy="1.54 0 0.77" />
       <geometry>
         <mesh filename="package://tesr_ros_cr3_pkg/meshes/base_gripper.stl" scale="0.001 0.001 0.001" />

Commit message: move back to same urdf not expand collision

File: cr3_ws/src/tesr_ros_cr3_pkg/urdf/cr3_robot_w_gripper_seperated.xacro (robot description, xacro)
@@ -66,5 +66,5 @@
       <origin xyz="0 0 0" rpy="0 0 0" />
       <geometry>
-        <mesh filename="package://tesr_ros_cr3_pkg/meshes/Link1.STL" scale="1.3 1.3 1.3"/>
+        <mesh filename="package://tesr_ros_cr3_pkg/meshes/Link1.STL" />
       </geometry>
     </collision>
@@ -91,7 +91,7 @@
     </visual>
     <collision>
-      <origin xyz="0.025 0.0 -0.025" rpy="0 0 0" />
-      <geometry>
-        <mesh filename="package://tesr_ros_cr3_pkg/meshes/Link2.STL" scale="1.1 1.3 1.3" />
+      <origin xyz="0 0 0" rpy="0 0 0" />
+      <geometry>
+        <mesh filename="package://tesr_ros_cr3_pkg/meshes/Link2.STL" />
       </geometry>
     </collision>
@@ -118,7 +118,7 @@
     </visual>
     <collision>
-      <origin xyz="0.025 0 0.0" rpy="0 0 0" />
-      <geometry>
-        <mesh filename="package://tesr_ros_cr3_pkg/meshes/Link3.STL" scale="1.1 1.5 1.5"/>
+      <origin xyz="0 0 0" rpy="0 0 0" />
+      <geometry>
+        <mesh filename="package://tesr_ros_cr3_pkg/meshes/Link3.STL" />
       </geometry>
     </collision>
@@ -147,5 +147,5 @@
       <origin xyz="0 0 0" rpy="0 0 0" />
       <geometry>
-        <mesh filename="package://tesr_ros_cr3_pkg/meshes/Link4.STL" scale="1.1 1.5 1.5"/>
+        <mesh filename="package://tesr_ros_cr3_pkg/meshes/Link4.STL" />
       </geometry>
     </collision>
@@ -174,5 +174,5 @@
       <origin xyz="0 0 0" rpy="0 0 0" />
       <geometry>
-        <mesh filename="package://tesr_ros_cr3_pkg/meshes/Link5.STL" scale="1.1 1.5 1.5"/>
+        <mesh filename="package://tesr_ros_cr3_pkg/meshes/Link5.STL" />
       </geometry>
     </collision>
@@ -201,5 +201,5 @@
       <origin xyz="0 0 0" rpy="0 0 0" />
       <geometry>
-        <mesh filename="package://tesr_ros_cr3_pkg/meshes/Link6.STL" scale="1 1 1"/>
+        <mesh filename="package://tesr_ros_cr3_pkg/meshes/Link6.STL" />
       </geometry>
     </collision>
@@ -226,5 +226,5 @@
     </visual>
     <collision>
-      <origin xyz="0.010 0.065 0.05" rpy="1.54 0 0.77" />
+      <origin xyz="0.053 0.035 0.05" rpy="1.54 0 0.77" />
       <geometry>
         <mesh filename="package://tesr_ros_cr3_pkg/meshes/base_gripper.stl" scale="0.001 0.001 0.001" />

Commit message: add collision cr3 and smach_place

File: cr3_ws/src/tesr_ros_cr3_pkg/urdf/cr3_robot_w_gripper_seperated.xacro (robot description, xacro)
@@ -129,5 +129,5 @@
     <child link="Link3" />
     <axis xyz="0 0 1" />
-    <limit lower="-3.14" upper="3.14" effort="1000" velocity="100" />
+    <limit lower="-2.70" upper="2.70" effort="1000" velocity="100" />
      <!-- <dynamics damping="${damping_value}" friction="${friction_value}"/> -->
   </joint>
@@ -174,5 +174,5 @@
       <origin xyz="0 0 0" rpy="0 0 0" />
       <geometry>
-        <mesh filename="package://tesr_ros_cr3_pkg/meshes/Link5.STL" />
+        <mesh filename="package://tesr_ros_cr3_pkg/meshes/Link5.STL" scale="1.1 1.3 1.3"/>
       </geometry>
     </collision>
