Commit message: fix fail at initial gazebo

File: panda_ws/src/franka_ros/franka_description/robots/panda_arm.xacro (robot description, xacro)
@@ -175,5 +175,5 @@
     <joint name="${arm_id}_joint4" type="revolute">
       <safety_controller k_position="100.0" k_velocity="40.0" soft_lower_limit="-3.0718" soft_upper_limit="-0.0698"/>
-      <origin rpy="${pi/2} 0 0" xyz="0.0825 0 0"/>
+      <origin rpy="${pi/2} ${-pi} 0" xyz="0.0825 0 0"/>
       <parent link="${arm_id}_link3"/>
       <child link="${arm_id}_link4"/>
