Commit message: add prism model, set gazebo paused at initial

File: panda_ws/src/franka_ros/franka_description/robots/hand.xacro (robot description, xacro)
@@ -71,5 +71,5 @@
       <axis xyz="0 -1 0"/>
       <limit effort="20" lower="0.0" upper="0.04" velocity="0.2"/>
-      <mimic joint="${ns}_finger_joint1" />
+      <!-- <mimic joint="${ns}_finger_joint1" /> -->
     </joint>
   </xacro:macro>

File: panda_ws/src/franka_ros/franka_description/robots/panda_arm.xacro (robot description, xacro)
@@ -175,5 +175,5 @@
     <joint name="${arm_id}_joint4" type="revolute">
       <safety_controller k_position="100.0" k_velocity="40.0" soft_lower_limit="-3.0718" soft_upper_limit="-0.0698"/>
-      <origin rpy="${pi/2} ${-pi} 0" xyz="0.0825 0 0"/>
+      <origin rpy="${pi/2} 0 0" xyz="0.0825 0 0"/>
       <parent link="${arm_id}_link3"/>
       <child link="${arm_id}_link4"/>

File: panda_ws/src/panda_moveit_config/config/hand.xacro (robot description, xacro)
@@ -12,5 +12,6 @@
       <link name="panda_rightfinger" />
       <joint name="panda_finger_joint1" />
-      <passive_joint name="panda_finger_joint2" />
+      <!-- <passive_joint name="panda_finger_joint2" /> -->
+      <joint name="panda_finger_joint2" />
     </group>
     <!--GROUP STATES: Purpose: Define a named state for a particular group, in terms of joint values. This is useful to define states like 'folded arms'-->

Commit message: adjust hand.xacro for easy grip, still fail

File: panda_ws/src/franka_ros/franka_description/robots/hand.xacro (robot description, xacro)
@@ -30,12 +30,53 @@
     </link>
     <link name="${ns}_leftfinger">
-      <visual>
+      <!-- <visual>
         <geometry>
           <mesh filename="package://franka_description/meshes/visual/finger.dae"/>
         </geometry>
       </visual>
+      <collision>
+        <geometry>
+          <mesh filename="package://franka_description/meshes/collision/finger.stl"/>
+        </geometry>
+      </collision> -->
+      <!-- contact infomatioin based on https://answers.gazebosim.org//question/9371/finger-contact-erp-cfm-kp-and-kd/-->
+      <visual>
+        <origin xyz="0 0 0.03" rpy="0 0 0" />
+        <geometry>
+          <box size="0.02 0.02 0.06"/>
+        </geometry>
+      </visual>
+      <collision>
+        <origin xyz="0 0 0.03" rpy="0 0 0" />
+        <max_contacts>10</max_contacts>
+        <geometry>
+          <box size="0.02 0.02 0.06"/>
+        </geometry>
+        <surface>
+          <friction>
+            <ode>
+              <mu>0.8</mu>
+              <mu2>0.8</mu2>
+            </ode>
+          </friction>
+          <bounce>
+            <restitution_coefficient>0.01</restitution_coefficient>
+            <threshold>0.01</threshold>
+          </bounce>
+          <contact>
+            <ode>
+              <max_vel>0.1</max_vel>
+              <soft_cfm>0.8</soft_cfm>
+              <soft_erp>0.8</soft_erp>
+              <kd>2500</kd>
+              <kp>10</kp>
+              <min_depth>0.001</min_depth>
+            </ode>
+          </contact>
+        </surface>
+      </collision>
       <!-- for simulation -->
       <inertial>
-        <origin xyz="0 0 0" rpy="0 0 0" />
+        <origin xyz="0 0 0.03" rpy="0 0 0" />
         <mass value="0.68" />
         <inertia ixx="0.1" ixy="0.0" ixz="0.0" iyy="0.1" iyz="0.0" izz="0.1" />
@@ -44,5 +85,5 @@
     </link>
     <link name="${ns}_rightfinger">
-      <visual>
+      <!-- <visual>
         <origin xyz="0 0 0" rpy="0 0 ${pi}"/>
         <geometry>
@@ -50,7 +91,48 @@
         </geometry>
       </visual>
+      <collision>
+        <origin xyz="0 0 0" rpy="0 0 ${pi}"/>
+        <geometry>
+          <mesh filename="package://franka_description/meshes/collision/finger.stl"/>
+        </geometry>
+      </collision> -->
+      <visual>
+        <origin xyz="0 0 0.03" rpy="0 0 ${pi}"/>
+        <geometry>
+          <box size="0.02 0.02 0.06"/>
+        </geometry>
+      </visual>
+      <collision>
+        <origin xyz="0 0 0.03" rpy="0 0 ${pi}"/>
+        <max_contacts>10</max_contacts>
+        <geometry>
+          <box size="0.02 0.02 0.06"/>
+        </geometry>
+        <surface>
+          <friction>
+            <ode>
+              <mu>0.8</mu>
+              <mu2>0.8</mu2>
+            </ode>
+          </friction>
+          <bounce>
+            <restitution_coefficient>0.01</restitution_coefficient>
+            <threshold>0.01</threshold>
+          </bounce>
+          <contact>
+            <ode>
+              <max_vel>0.1</max_vel>
+              <soft_cfm>0.8</soft_cfm>
+              <soft_erp>0.8</soft_erp>
+              <kd>2500</kd>
+              <kp>10</kp>
+              <min_depth>0.001</min_depth>
+            </ode>
+          </contact>
+        </surface>
+      </collision>
       <!-- for simulation -->
       <inertial>
-        <origin xyz="0 0 0" rpy="0 0 0" />
+        <origin xyz="0 0 0.03" rpy="0 0 ${pi}"/>
         <mass value="0.68" />
         <inertia ixx="0.1" ixy="0.0" ixz="0.0" iyy="0.1" iyz="0.0" izz="0.1" />
@@ -61,14 +143,14 @@
       <parent link="${ns}_hand"/>
       <child link="${ns}_leftfinger"/>
-      <origin xyz="0 0 0.0584" rpy="0 0 0"/>
+      <origin xyz="0 0.018 0.0584" rpy="0 0 0"/>
       <axis xyz="0 1 0"/>
-      <limit effort="20" lower="0.0" upper="0.04" velocity="0.2"/>
+      <limit effort="20" lower="0.00" upper="0.04" velocity="0.2"/>
     </joint>
     <joint name="${ns}_finger_joint2" type="prismatic">
       <parent link="${ns}_hand"/>
       <child link="${ns}_rightfinger"/>
-      <origin xyz="0 0 0.0584" rpy="0 0 0"/>
+      <origin xyz="0 -0.018 0.0584" rpy="0 0 0"/>
       <axis xyz="0 -1 0"/>
-      <limit effort="20" lower="0.0" upper="0.04" velocity="0.2"/>
+      <limit effort="20" lower="0.00" upper="0.04" velocity="0.2"/>
       <!-- <mimic joint="${ns}_finger_joint1" /> -->
     </joint>
